File: SGR/SGR.kicad_pcb (KiCad board)
At the start: 2 copper layers, 20 x 20 mm, 14 parts, among them U1 MCP1642B-50I/MS

Commit message: Add files via upload
Routing:
- removed copper zone on B.Cu, net /SW
Other:
- board text added: "@Jackv_makes"
Changed lines of the file:
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@@
 			(drillshape 0)
 			(scaleselection 1)
-			(outputdirectory "C:/Users/Jacks/Downloads/POG/New_POG/GTR34/V1.1/")
+			(outputdirectory "C:/Users/Jacks/Downloads/POG/SGR/V1.1/")
 		)
 	)
@@
 		)
 	)
+	(gr_text "@Jackv_makes"
+		(at 146.175 81.35 0)
+		(layer "B.SilkS")
+		(effects
+			(font
+				(size 1 1)
+				(thickness 0.2)
+				(bold yes)
+			)
+			(justify left bottom mirror)
+		)
+	)
 	(gr_text "V1.1"
 		(at 133.5 81.5 0)
@@
 	)
 	(zone
+		(net 6)
+		(net_name "/SW")
+		(layer "F.Cu")
+		(hatch edge 0.5)
+		(priority 3)
+		(connect_pads yes
+			(clearance 0.2)
+		)
+		(min_thickness 0.2)
+		(filled_areas_thickness no)
+		(fill yes
+			(thermal_gap 0.3)
+			(thermal_bridge_width 0.3)
+		)
+		(polygon
+			(pts
+				(xy 138.775 83.375) (xy 138.775 89.5) (xy 139.8 89.5) (xy 140 89.5) (xy 140 83.375)
+			)
+		)
+	)
+	(zone
 		(net 4)
 		(net_name "/GBVDD")
@@
 			)
 		)
-	)
-	(zone
-		(net 6)
-		(net_name "/SW")
-		(layers "F&B.Cu")
-		(hatch edge 0.5)
-		(priority 3)
-		(connect_pads yes
-			(clearance 0.2)
-		)
-		(min_thickness 0.2)
-		(filled_areas_thickness no)
-		(fill yes
-			(thermal_gap 0.3)
-			(thermal_bridge_width 0.3)
-		)
-		(polygon
-			(pts
-				(xy 138.775 83.375) (xy 138.775 89.5) (xy 139.8 89.5) (xy 140 89.5) (xy 140 83.375)
-			)
-		)

Commit message: Add files via upload
Parts:
- removed GBVCC, GBVDD, GND: ~, TestPoint:TestPoint_Pad_D2.5mm
Routing:
- net GND: vias 3 -> 0
- net /GBVDD: vias 3 -> 0
- net /GBVCC: vias 3 -> 0
